File: artnet-led-controller/artnet-led-controller.kicad_sch (KiCad schematic)
At the start: 71 parts, among them J1 USB4125-GF-A, J10 SWD_DEBUG, J2 HR911105A, J3 VBAT JST-PH-2, J5 LED_OUT_1, J6 LED_OUT_2, J7 LED_OUT_3, J8 LED_OUT_4, J9 OLED_SSD1306, SW1 BTN1, SW2 BTN2, SW3 RESET, U1 RP2040, U2 W25Q16JVSSIQ, U3 W5500, U4 SN74AHCT125, U5 TP4056, U6 MT3608, U7 AMS1117-3.3, Y1 12MHz, Y2 25MHz

Commit message: Redesign controller around RP2354A
Parts:
- removed C1: 100nF, Capacitor_SMD:C_0402_1005Metric, symbol C
- removed U1: RP2040, Package_DFN_QFN:QFN-56-1EP_7x7mm_P0.4mm_EP3.2x3.2mm, symbol RP2040
- removed U2: W25Q16JVSSIQ, Package_SO:SOIC-8_3.9x4.9mm_P1.27mm, symbol W25Q16JV
- added C10, C51, C7, C9: 4.7uF, Capacitor_SMD:C_0402_1005Metric, symbol C
- added C52, C8: 100nF, Capacitor_SMD:C_0402_1005Metric, symbol C
- added D1: SS14, Diode_SMD:D_SOD-123, symbol D_Schottky
- added L2: 3.3uH, Inductor_SMD:L_0805_2012Metric, symbol L
- added R23: 33, Resistor_SMD:R_0402_1005Metric, symbol R
- added R24: 1k, Resistor_SMD:R_0402_1005Metric, symbol R
- added SW4: BOOTSEL, Button_Switch_SMD:SW_Push_1P1T_NO_CK_KSC7xxJ, symbol SW_Push
- added U1: RP2354A, Package_DFN_QFN:QFN-60-1EP_7x7mm_P0.4mm_EP3.4x3.4mm, symbol RP2354A
- C43: value 1uF -> 100nF; LCSC C52923 -> C14663
- C46: value 100nF -> 4.7uF; LCSC C14663 -> C19712
- C49: value 4.7uF -> 100nF; LCSC C19712 -> C14663
- J1: footprint Connector_USB:USB_C_Receptacle_GCT_USB4125_1x_1614 -> Connector_USB:USB_C_Receptacle_GCT_USB4125-xx-x_6P_TopMnt_Horizontal
- J2: footprint Connector_RJ:RJ45_Amphenol_54602-x08_Horizontal -> Connector_RJ:RJ45_Hanrun_HR911105A_Horizontal
- SW1, SW2, SW3: footprint Button_Switch_SMD:SW_Push_1P1T_NO_Vertical_Straight_PadInPin_CK_KSC741J -> Button_Switch_SMD:SW_Push_1P1T_NO_CK_KSC7xxJ
Connections:
- net BTN1: now also U1.57 (QSPI_SD0)
- net BTN2: now also U1.56 (QSPI_SCLK)
- net I2C_SCL: now also U1.19 (GPIO15)
- net I2C_SDA: now also U1.21 (XIN)
- net LED1_DATA_3V3: now also U1.26 (RUN)
- net LED2_DATA_3V3: now also U1.51 (USB_DM)
- net LED3_DATA_3V3: now also U1.52 (USB_DP)
- net LED4_DATA_3V3: now also U1.22 (XOUT)
- net MT3608_SW: now also D1.2 (K); no longer J5.1 (Pin1), J6.1 (Pin1), J7.1 (Pin1), J8.1 (Pin1), R1.2, U6.6 (NC), U7.4 (VOUT2)
- net RP_RUN: now also U1.2 (GPIO0)
- net RP_XIN: now also U1.7 (GPIO4)
- net RP_XOUT: now also U1.5 (GPIO3)
- net SPI_MOSI: now also U1.55 (QSPI_SD3)
- net USB_DM: now also U1.3 (GPIO1)
- net USB_DP: now also U1.4 (GPIO2)
- net VCC3V3: now also R23.2
- net W5500_INT: now also U1.58 (QSPI_SD2)
- net W5500_RST: now also U1.59 (QSPI_SD1)
- new net USB_BOOT: R24.2, U1.36 (GPIO24)
- new net USB_BOOT_SW: R24.1, SW4.1 (A)
- new net VCC5V: D1.1 (A), J5.1 (Pin1), J6.1 (Pin1), J7.1 (Pin1), J8.1 (Pin1), R1.2, U6.6 (NC), U7.4 (VOUT2)
- new net VREG_1V1: C10.2, C7.2, C9.2, L2.1
- new net VREG_AVDD: C8.2, R23.1
- new net VREG_LX: L2.2
- no-connect marks 29 -> 34
