File: artnet-led-controller/artnet-led-controller.kicad_sch (KiCad schematic)
At the start: 80 parts, among them J1 USB4125-GF-A, J10 SWD_DEBUG, J2 HR911105A, J3 VBAT JST-PH-2, J5 LED_OUT_1, J6 LED_OUT_2, J7 LED_OUT_3, J8 LED_OUT_4, J9 OLED_SSD1306, SW1 BTN1, SW2 BTN2, SW3 RESET, SW4 BOOTSEL, U1 RP2354A, U3 W5500, U4 SN74AHCT125, U5 TP4056, U6 MT3608, U7 AMS1117-3.3, Y1 12MHz, Y2 25MHz

Commit message: Add netlist extraction and PCB pad net assignment
gen_schematic.py now exports netlist.json mapping each ref to its
pad-to-net assignments. gen_pcb.py loads this and injects (net N "name")
into every pad block so the board is routable with freerouting.
Also fixes pin_ep sign bug (cy+py -> cy-py) in schematic generator.

Co-Authored-By: Claude Sonnet 4.6 <noreply@anthropic.com>
Connections:
- net BTN1: now also U1.34 (GPIO22); no longer U1.57 (QSPI_SD0)
- net BTN2: now also U1.35 (GPIO23); no longer U1.56 (QSPI_SCLK)
- net ETH_CT1: now also J2.8 (CT1); no longer J2.9 (CT2)
- net ETH_CT2: now also J2.9 (CT2); no longer J2.8 (CT1)
- net ETH_RXN: now also U3.13 (RXN); no longer U3.6 (AVCCRST)
- net ETH_RXP: now also J2.13 (MDO+), U3.14 (RXP); no longer J2.15 (LINK_LED), U3.29 (RSVD6)
- net ETH_TXN: now also J2.12 (MDI-), U3.12 (TXN); no longer J2.16 (ACT_LED), U3.30 (RSVD7)
- net ETH_TXP: now also J2.11 (MDI+), U3.11 (TXP); no longer J2.17 (SHIELD), U3.31 (RSVD8)
- net I2C_SCL: now also J9.3 (Pin3), U1.8 (GPIO5); no longer J9.1 (Pin1), U1.19 (GPIO15)
- net I2C_SDA: now also J9.4 (Pin4), U1.7 (GPIO4); no longer U1.21 (XIN)
- net LED1_DATA_3V3: now also U1.2 (GPIO0), U4.2 (A1); no longer U1.26 (RUN), U4.9 (/OE_C)
- net LED1_DATA_5V: now also U4.3 (Y1); no longer U4.11 (Y4)
- net LED2_DATA_3V3: now also U1.3 (GPIO1), U4.5 (A2); no longer U1.51 (USB_DM), U4.4 (/OE_B)
- net LED2_DATA_5V: now also U4.6 (Y2); no longer U4.8 (Y3)
- net LED3_DATA_3V3: now also U1.4 (GPIO2), U4.10 (A3); no longer U1.52 (USB_DP), U4.1 (/OE_A)
- net LED3_DATA_5V: now also U4.8 (Y3); no longer U4.6 (Y2)
- net LED4_DATA_3V3: now also U1.5 (GPIO3), U4.13 (A4); no longer U1.22 (XOUT), U4.12 (/OE_D)
- net LED4_DATA_5V: now also U4.11 (Y4); no longer U4.3 (Y1)
- net MT3608_FB: now also U6.4 (FB); no longer U6.5 (SW)
- net MT3608_SW: now also U6.5 (SW); no longer D1.2 (K), L1.1, U6.4 (FB)
- net RP_RUN: now also U1.26 (RUN); no longer U1.2 (GPIO0)
- net RP_XIN: now also U1.21 (XIN); no longer U1.7 (GPIO4)
- net RP_XOUT: now also U1.22 (XOUT); no longer U1.5 (GPIO3)
- net SPI_CS: now also U1.28 (GPIO17), U3.24 (/SCSn); no longer U3.3 (RSVD3)
- net SPI_MISO: now also U1.27 (GPIO16), U3.21 (MISO); no longer U3.5 (EXRES1)
- net SPI_MOSI: now also U1.31 (GPIO19), U3.22 (MOSI); no longer U1.55 (QSPI_SD3), U3.17 (RSVD5)
- net SPI_SCK: now also U1.29 (GPIO18), U3.23 (SCLK); no longer U3.4 (RSVD4)
- net STDBY_STAT: now also U5.7 (/STDBY); no longer U5.5 (BAT)
- net SWCLK: now also J10.1 (Pin1), U1.24 (SWCLK); no longer J10.3 (Pin3)
- net SWDIO: now also U1.25 (SWDIO)
- net TP4056_PROG: now also J1.A1 (VBUS), J1.B1 (VBUS2), U5.4 (VCC); no longer J1.A12 (GND), J1.B5 (CC2), U5.8 (TE)
- net USB_BOOT: now also U1.60 (QSPI_SS); no longer U1.36 (GPIO24)
- net USB_CC1: now also J1.A5 (CC1); no longer J1.A7 (D-)
- net USB_CC2: now also J1.B5 (CC2); no longer J1.A1 (VBUS)
- net USB_DM: now also J1.A7 (D-), U1.51 (USB_DM); no longer J1.A5 (CC1), U1.3 (GPIO1)
- net USB_DP: now also U1.52 (USB_DP); no longer U1.4 (GPIO2)
- net VBAT: now also J3.1 (Pin1), U5.5 (BAT), U6.1 (IN); no longer J3.2 (Pin2), U5.7 (/STDBY), U6.2 (GND)
- net VCC3V3: now also U7.4 (VOUT2); no longer U7.3 (VIN)
- net VCC5V: now also J5.3 (Pin3), J6.3 (Pin3), J7.3 (Pin3), J8.3 (Pin3), U6.3 (EN), U7.3 (VIN); no longer J5.1 (Pin1), J6.1 (Pin1), J7.1 (Pin1), J8.1 (Pin1), U6.6 (NC), U7.4 (VOUT2)
- net VREG_1V1: now also U1.23 (DVDD2), U1.39 (DVDD3), U1.50 (VREG_FB), U1.6 (DVDD1)
- net VREG_AVDD: now also U1.46 (VREG_AVDD)
- net VREG_LX: now also U1.48 (VREG_LX)
- net W5500_EXRES0: now also U3.10 (EXRES0); no longer U3.16 (XTAL2)
- net W5500_EXRES1: now also U3.5 (EXRES1), U3.6 (AVCCRST); no longer U3.13 (RXN), U3.21 (MISO)
- net W5500_INT: now also U1.32 (GPIO20), U3.27 (/INTn); no longer U1.58 (QSPI_SD2), U3.2 (RSVD2)
- net W5500_RCLK: now also U3.9 (RCLK); no longer U3.15 (XTAL1)
- net W5500_RST: now also U1.33 (GPIO21), U3.28 (/RSTn); no longer U1.59 (QSPI_SD1), U3.1 (RSVD1)
- net W5_VDD: now also U3.26 (VDD); no longer U3.32 (GND2)
- net W5_XTAL1: now also U3.15 (XTAL1); no longer U3.9 (RCLK)
- net W5_XTAL2: now also U3.16 (XTAL2); no longer U3.10 (EXRES0)
- new net VBOOST_RAW: D1.2 (K), L1.1
